File: Personal_Projects/PCB/BUCK_V1/BUCK_V1.kicad_pcb (KiCad board)
At the start: 2 copper layers, 10 parts, among them J1 Conn_01x03_Socket, U1 AP62150WU

Commit message: lab7
Parts:
- moved L1 20.8 mm to (134.5, 60.0)
- moved C1 16.0 mm to (130.0, 63.6)
- moved C2 13.3 mm to (142.5, 59.0), turned to 0 degrees
- moved U1 7.76 mm to (144.0, 66.0)
- moved L2 6.40 mm to (139.5, 75.0)
- moved R2 5.10 mm to (150.0, 52.0)
Connections:
- J1 pad 1: unconnected-(J1-Pin_1-Pad1) -> +12V
- J1 pad 2: unconnected-(J1-Pin_2-Pad2) -> GND
- J1 pad 3: unconnected-(J1-Pin_3-Pad3) -> /Vout
Routing:
- net /Vout: track 0.00 -> 60.0 mm
- net +12V: track 0.00 -> 33.4 mm
- net Net-(U1-SW): track 0.00 -> 19.2 mm
- net Net-(L1-Pad2): track 0.00 -> 15.8 mm
- net Net-(U1-FB): track 9.00 -> 21.7 mm
- net Net-(U1-BST): track 0.00 -> 6.98 mm
Other:
- board outline added: 44 x 36 mm
- board text added: "5V Buck Converter"
- board text added: "GND"
- board text added: "Gavin Simpson"
- board text added: "Vin"
- board text added: "Vout"
